Commit message: Localization TF corrections

File: realsense_explorer_description/urdf/realsense_bot.urdf (robot description, URDF)
Before this commit: robot realsense_explorer, 22 links, 21 joints
Links:
- removed link base_footprint
- removed link imu_link
- removed link link_left_wheel
- removed link link_right_wheel
- removed link robot_base
Joints:
- removed joint base_joint
- removed joint chasis_to_rbot
- removed joint imu_joint
- removed joint joint_left_wheel
- removed joint joint_right_wheel

File: realsense_explorer_description/urdf/realsense_explorer.urdf.xacro (robot description, xacro)
@@ -4,5 +4,5 @@
   <xacro:arg name="add_plug" default="false" />
   <xacro:arg name="use_mesh" default="true" />
-  <xacro:include filename="$(find realsense_bot)/urdf/realsense_bot.urdf.xacro" />
+  <xacro:include filename="$(find realsense_explorer_description)/urdf/realsense_bot.urdf.xacro" />
   <material name="invisible">
     <color rgba="0 0 0 0"/>
@@ -10,4 +10,7 @@
   <material name="green">
     <color rgba="0 1 0 1"/>
+  </material>
+  <material name="grey">
+    <color rgba="0.9 0.9 0.9 1"/>
   </material>
 <link name="base_footprint"/>
@@ -18,4 +21,5 @@
         <mesh scale="0.001 0.001 0.001" filename="package://realsense_explorer_description/meshes/robot_chassis.STL"/>
       </geometry>
+      <material name="grey"/>
     </visual>
       <collision>
@@ -33,5 +37,5 @@
   <joint name="chasis_to_rbot" type="fixed">
     <parent link="robot_base"/>
-    <child link="world"/>
+    <child link="rbot_base"/>
     <origin xyz="-0.09 0 0.13787" rpy="0 0 0"/>
   </joint>
