Commit message: Imu Frames Update

File: realsense_explorer_description/urdf/realsense_explorer.urdf (robot description, URDF)
Before this commit: robot realsense_explorer, 21 links, 20 joints
Links:
- added link imu_link; visual box size=0.015 0.026 0.001
Joints:
- added joint imu_joint: type fixed, parent robot_base, child imu_link, origin xyz=0.114 0 0.05 rpy=0 0 0

File: realsense_explorer_description/urdf/realsense_explorer.urdf.xacro (robot description, xacro)
@@ -5,10 +5,9 @@
   <xacro:arg name="use_mesh" default="true" />
   <xacro:include filename="$(find realsense_bot)/urdf/realsense_bot.urdf.xacro" />
-  <!-- <link name="base_link" />
-  <xacro:realsense_bot parent="base_link" use_nominal_extrinsics="true" add_plug="false" use_mesh="true">
-    <origin xyz="0 0 0" rpy="0 0 0"/>
-  </xacro:realsense_bot> -->
   <material name="invisible">
     <color rgba="0 0 0 0"/>
+  </material>
+  <material name="green">
+    <color rgba="0 1 0 1"/>
   </material>
 <link name="base_footprint"/>
@@ -83,4 +82,17 @@
   <joint_properties damping="1.0" friction="1.0" />
 </joint>
+  <link name="imu_link">
+    <visual>
+      <geometry>
+        <box size="0.015 0.026 0.001"/>
+      </geometry>
+      <material name="green"/>
+    </visual>
+  </link>
+<joint name="imu_joint" type="fixed">
+  <origin rpy="0 0 0" xyz="0.114 0 0.05"/>
+  <child link="imu_link" />
+  <parent link="robot_base"/>
+</joint>
 <transmission name="right_wheel_transmission">
   <type>transmission_interface/SimpleTransmission</type>

Commit message: Gazebo Support WIP

File: realsense_explorer_description/urdf/realsense_explorer.urdf (robot description, URDF)
Before this commit: robot realsense_explorer, 22 links, 21 joints
Links:
- removed link U_Link
- removed link base_footprint
- removed link base_link
- removed link camera_bottom_screw_frame
- removed link camera_color_frame
- removed link camera_color_optical_frame
- removed link camera_depth_frame
- removed link camera_depth_optical_frame
- removed link camera_infra1_frame
- removed link camera_infra1_optical_frame
- removed link camera_infra2_frame
- removed link camera_infra2_optical_frame
- removed link camera_link
- removed link imu_link
- removed link link_left_wheel
- removed link link_right_wheel
- removed link rbot_base
- removed link servo_bottom
- removed link servo_mid
- removed link servo_up
- removed link up_mount
- added link camera_mount_link, mass 0.0417767995564032; collision mesh filename=package://realsense_explorer/meshes/camera_mount_link.STL; visual mesh filename=package://realsense_explorer/meshes/camera_mount_link.STL
- added link left_wheel_link, mass 0.446655935524129; collision mesh filename=package://realsense_explorer/meshes/left_wheel_link.STL; visual mesh filename=package://realsense_explorer/meshes/left_wheel_link.STL
- added link long_u_link, mass 0.0213372016014766; collision mesh filename=package://realsense_explorer/meshes/long_u_link.STL; visual mesh filename=package://realsense_explorer/meshes/long_u_link.STL
- added link mid_servo_link, mass 0.0977262710445392; collision mesh filename=package://realsense_explorer/meshes/mid_servo_link.STL; visual mesh filename=package://realsense_explorer/meshes/mid_servo_link.STL
- added link right_wheel_link, mass 0.446655935524129; collision mesh filename=package://realsense_explorer/meshes/right_wheel_link.STL; visual mesh filename=package://realsense_explorer/meshes/right_wheel_link.STL
- link robot_base: mass None -> 3.84203102747016; geometry collision mesh filename=package://realsense_explorer/meshes/robot_base.STL; visual mesh filename=package://realsense_explorer/meshes/robot_base.STL
Joints:
- removed joint Joint_1
- removed joint Joint_2
- removed joint Joint_3
- removed joint base_joint
- removed joint base_to_Servo_B
- removed joint camera_color_joint
- removed joint camera_color_optical_joint
- removed joint camera_depth_joint
- removed joint camera_depth_optical_joint
- removed joint camera_infra1_joint
- removed joint camera_infra1_optical_joint
- removed joint camera_infra2_joint
- removed joint camera_infra2_optical_joint
- removed joint camera_joint
- removed joint camera_link_joint
- removed joint chasis_to_rbot
- removed joint imu_joint
- removed joint joint_left_wheel
- removed joint joint_right_wheel
- removed joint mount_to_camera
- removed joint servo_mid_to_servo_up
- added joint camera_mount_joint: type continuous, parent mid_servo_link, child camera_mount_link, origin xyz=0.0378975953962198 -0.00642581350278899 -0.0210000000000001 rpy=-1.57079632679501 -1.56018827190785 -0.791795520542192, axis 0 0 1
- added joint left_wheel_joint: type continuous, parent robot_base, child left_wheel_link, origin xyz=0.033161 0.07075 0.055 rpy=-1.5708 0 0, axis 0 0 1
- added joint long_u_joint: type continuous, parent robot_base, child long_u_link, origin xyz=-0.0457291882084462 -0.01125 0.19927 rpy=0 0 1.5707963267949, axis 0 0 1
- added joint mid_joint_link: type continuous, parent long_u_link, child mid_servo_link, origin xyz=0 0 0.05 rpy=-1.5707963267949 -1.54960030838858 -1.57079632679489, axis 0 0 1
- added joint right_wheel_joint: type continuous, parent robot_base, child right_wheel_link, origin xyz=0.033161 -0.07075 0.055 rpy=-1.5708 0 0, axis 0 0 1
