Commit message: Realsense Plugin Update

File: realsense_explorer_description/urdf/realsense_explorer_gazebo.urdf.xacro (robot description, xacro)
@@ -6,12 +6,8 @@
   <xacro:arg name="use_mesh" default="true" />
   <xacro:include filename="$(find realsense2_description)/urdf/_d435.urdf.xacro" />
-<sensor_d435 parent="camera_mount_link">
-  <origin xyz="0 0 0" rpy="0 0 0"/>
-</sensor_d435>
-<!-- <joint name="mount_to_camera" type="fixed">
-  <parent link="camera_mount_link"/>
-  <child link="camera_link"/>
-  <origin xyz="0.03 0 0.02" rpy="0 -0.785 0"/>
-</joint> -->
+  <xacro:arg name="use_nominal_extrinsics" default="true"/>
+<xacro:sensor_d435 parent="camera_mount_link" use_nominal_extrinsics="$(arg use_nominal_extrinsics)">
+  <origin xyz="-0.0031452 -0.0089594 0.063032" rpy="0 -0.8002 -1.5814"/>
+</xacro:sensor_d435>
   <gazebo>
     <plugin name="gazebo_ros_control" filename="libgazebo_ros_control.so">
@@ -141,6 +137,5 @@
   </sensor>
 </gazebo>
-</robot>
-  <!-- <gazebo reference="camera_color_frame">
+  <gazebo reference="camera_color_frame">
     <sensor name="color" type="camera">
       <pose frame="">0 0 0 0 0 0</pose>
@@ -265,6 +260,6 @@
         <pointCloudCutoffMax>10</pointCloudCutoffMax>
       </plugin>
-  </gazebo> -->
-  <!-- <gazebo reference="camera_gyro_frame">
+  </gazebo>
+  <gazebo reference="camera_gyro_frame">
     <gravity>true</gravity>
     <sensor name="imu_sensor" type="imu">
@@ -283,3 +278,4 @@
       <pose>0 0 0 0 0 0</pose>
     </sensor>
-  </gazebo> -->
+  </gazebo>
+</robot>
